Commit message: Update to v1.0.0

File: marmorf_description/urdf/marmorf.urdf (robot description, URDF)
Before this commit: robot marmorf_urdf, 12 links, 11 joints
Joints:
- joint imu_joint: origin xyz=0.0 -0.1 0.0 rpy=-0.0036488 0.0047929 -0.002592 -> xyz=0.0 -0.1 0.0 rpy=-0.0036488 0.0047929 -1.57

File: marmorf_description/urdf/marmorf.urdf.xacro (robot description, xacro)
@@ -41,5 +41,5 @@
     <link name="imu_link"/>
     <joint name="imu_joint" type="fixed">
-      <origin xyz="0.0 0.0 0.0" rpy="0 0 0" />
+      <origin xyz="0.0 0.0 0.0" rpy="0 0 -1.57" />
       <parent link="marmorf_link" />
       <child link="imu_link" />
